Commit message: TA2 v0.9 - Hopefully the last version in terms of code. Only missing data for offline analysis.

File: src/TA2/gazebo_factory/urdf/tbox/tbox.urdf.xacro (robot description, xacro)
@@ -53,5 +53,5 @@
       <inertial>
         <origin xyz="0.0 0.0 ${boxh/2+legh}" rpy="0.0 0.0 0.0"/>
-        <mass value="0.5"/>
+        <mass value="2.0"/>
         <inertia ixx="0.005" ixy="0" ixz="0" iyy="0.005" iyz="0" izz="0.005"/>
       </inertial>
@@ -74,8 +74,12 @@
     <gazebo reference="${name}_base_link">
       <material>Gazebo/FlatBlack</material><!--youbot/DarkGrey-->
-      <mu1>0.5</mu1>
+ <!--     <mu1>0.5</mu1>
       <mu2>50.0</mu2>
       <kp>100000000.0</kp>
-      <kd>1.0</kd>
+      <kd>1.0</kd>-->
+      <kp>1000000.0</kp>
+      <kd>100.0</kd>
+      <mu1>500.0</mu1>
+      <mu2>500.0</mu2>
     </gazebo>
     <!-- Add left front leg -->

File: src/TA2/pioneer3dx_description/urdf/forklift/forklift.urdf.xacro (robot description, xacro)
@@ -8,5 +8,5 @@
   <xacro:property name="bw" value=".2" /> <!-- Base width -->
   <xacro:property name="bt" value=".06" /> <!-- Base thickness -->
-  <xacro:property name="sbf" value=".12" /> <!-- Space between fingers -->
+  <xacro:property name="sbf" value=".09" /> <!-- Space between fingers -->
   <xacro:property name="bfl" value=".2" /> <!-- Bottom finger length -->
   <xacro:property name="bft" value=".01" /> <!-- Bottom finger thickness -->
@@ -47,8 +47,12 @@
     <gazebo reference="bottom_${suffix}">
       <material value="Gazebo/Blue"/>
-      <mu1>0.5</mu1>
+<!--      <mu1>0.5</mu1>
       <mu2>50.0</mu2>
       <kp>100000000.0</kp>
+      <kd>1.0</kd>-->
+      <kp>1000000.0</kp>
       <kd>1.0</kd>
+      <mu1>500.0</mu1>
+      <mu2>500.0</mu2>
     </gazebo>
     <!-- Attach bottom finger to support -->
@@ -161,10 +165,10 @@
       <child link="${name}_fingers_support_link"/>
       <axis xyz="0 0 1"/>
-      <limit effort="100.0" lower="0.0" upper="10.08" velocity="0.3"/>
-<!--      <stopKd value="0.0" />
+      <limit effort="1000.0" lower="0.0" upper="10.08" velocity="0.2"/>
+      <stopKd value="0.0" />
       <stopKp value="0.0" />
       <fudgeFactor value="1.0" />
       <provideFeedback value="true"/>
-      <dynamics damping="10" />-->
+      <dynamics damping="10" />
     </joint>
     <transmission name="${name}_link_trans">

File: src/TA2/pioneer3dx_description/urdf/pioneer3dx/pioneer3dx.xacro (robot description, xacro)
@@ -10,5 +10,5 @@
     <inertial>
       <origin xyz="0 0 0.16"/>
-      <mass value="5.67"/>
+      <mass value="10.0"/>
       <inertia ixx="0.07" ixy="0" ixz="0" iyy="08" iyz="0" izz="0.10"/>
     </inertial>
@@ -29,5 +29,5 @@
   <link name="castor">
     <inertial>
-      <mass value="0.1"/>
+      <mass value="0.5"/>
       <origin xyz="-0.2 0 0.04"/>
       <inertia ixx="0.01" ixy="0.0" ixz="0.0" iyy="0.01" iyz="0" izz="0.01"/>

File: src/TA2/pioneer3dx_description/urdf/pioneer3dx/pioneer3dx_hokuyo_urg_camera.xacro (robot description, xacro)
@@ -17,5 +17,5 @@
     <xacro:include filename="$(find pioneer3dx_description)/urdf/sensors/gz_camera.xacro"/>
     <xacro:gz_camera parent="base_link" topic="/p3dx/camera_front">
-      <origin xyz="0.240 0.0 0.272" rpy="0 0 0"/>
+      <origin xyz="0.240 0.0 0.20" rpy="0 0 0"/>
     </xacro:gz_camera>
     <!-- Forklift -->

File: src/TA2/pioneer3dx_description/urdf/sensors/gz_camera.xacro (robot description, xacro)
@@ -49,12 +49,12 @@
             <far>300</far>
           </clip>
-<!--           <noise> -->
-<!--             <type>gaussian</type> -->
+          <noise>
+            <type>gaussian</type>
             <!-- Noise is sampled independently per pixel on each frame.
                 That pixel's noise value is added to each of its color
                   channels, which at that point lie in the range [0,1]. -->
-<!--             <mean>0.0</mean> -->
-<!--             <stddev>0.007</stddev> -->
-<!--           </noise> -->
+            <mean>0.0</mean>
+            <stddev>0.007</stddev>
+          </noise>
         </camera>
         <plugin name="camera_controller" filename="libgazebo_ros_camera.so">
