Commit message: Saving some minor changes, before a big updated on the forklift.

File: src/TA2/pioneer3dx_description/urdf/forklift/forklift.urdf.xacro (robot description, xacro)
@@ -23,10 +23,10 @@
     <link name="bottom_${suffix}">
       <inertial>
-        <origin xyz="${tft/2+bfl/2} ${reflect*(sbf/2+bfw/2)} ${-tfh/3}" rpy="0.0 ${M_PI/2+bfr} 0.0"/>
-        <mass value="0.1"/>
-        <inertia ixx="0.001" ixy="0" ixz="0" iyy="0.001" iyz="0" izz="0.001"/>
-      </inertial>
-      <collision name="collision">
-        <origin xyz="${tft/2+bfl/2} ${reflect*(sbf/2+bfw/2)} ${-tfh/3}" rpy="0.0 ${M_PI/2+bfr} 0.0"/>
+        <origin xyz="${tft/2+bfl/2} ${reflect*(sbf/2+bfw/2)} ${-tfh/3+bft/2}" rpy="0.0 ${M_PI/2+bfr} 0.0"/>
+        <mass value="0.1"/>
+        <inertia ixx="0.001" ixy="0" ixz="0" iyy="0.001" iyz="0" izz="0.001"/>
+      </inertial>
+      <collision name="collision">
+        <origin xyz="${tft/2+bfl/2} ${reflect*(sbf/2+bfw/2)} ${-tfh/3+bft/2}" rpy="0.0 ${M_PI/2+bfr} 0.0"/>
         <geometry>
            <box size="${bft} ${bfw} ${bfl}"/>

Commit message: Minor change to the forklift to improve its functioning.

File: src/TA2/pioneer3dx_description/urdf/forklift/forklift.urdf.xacro (robot description, xacro)
@@ -8,8 +8,8 @@
   <xacro:property name="bw" value=".2" /> <!-- Base width -->
   <xacro:property name="bt" value=".06" /> <!-- Base thickness -->
-  <xacro:property name="sbf" value=".09" /> <!-- Space between fingers -->
+  <xacro:property name="sbf" value=".10" /> <!-- Space between fingers -->
   <xacro:property name="bfl" value=".2" /> <!-- Bottom finger length -->
   <xacro:property name="bft" value=".01" /> <!-- Bottom finger thickness -->
-  <xacro:property name="bfw" value=".02" /> <!-- Bottom finger width -->
+  <xacro:property name="bfw" value=".03" /> <!-- Bottom finger width -->
   <xacro:property name="bfr" value="-.05" /> <!-- Bottom finger rotation -->
   <xacro:property name="tfh" value=".14" /> <!-- Top finger height -->
